Commit message: Change some urdf files making it could support multi robot tf publishing.

File: urdf/common/radar.urdf.xacro (robot description, xacro)
@@ -2,14 +2,13 @@
 <robot xmlns:xacro="http://www.ros.org/wiki/xacro" name="radar">
     <xacro:include filename="$(find sct_description)/urdf/common/inertia_utils.urdf.xacro"/>
-    <xacro:macro name="RADAR" params="connected_to radar_name use_sim name_space xyz:='0 0 0' rpy:='0 0 0' ">
-        <xacro:arg name="ns" default="${name_space}"/>
+    <xacro:macro name="RADAR" params="connected_to use_sim name_space xyz:='0 0 0' rpy:='0 0 0' ">
         <!-- Radar is fixed to the base link -->
-        <joint name="${radar_name}_joint" type="fixed">
+        <joint name="${name_space}_radar_joint" type="fixed">
             <origin xyz="${xyz}" rpy="${rpy}"/>
             <parent link="${connected_to}"/>
-            <child link="${radar_name}_link"/>
+            <child link="${name_space}_radar_link"/>
         </joint>
         <!-- Radar link -->
-        <link name="${radar_name}_link">
+        <link name="${name_space}_radar_link">
             <xacro:cylinder_inertial_matrix m="0.1" r="0.03" h="0.05"/>
             <visual>
@@ -29,13 +28,10 @@
             </material>
         </link>
-        <gazebo reference="${radar_name}">
-            <material>Gazebo/Orange</material>
-        </gazebo>
-        <gazebo reference="${radar_name}_joint">
+        <gazebo reference="radar_joint">
             <disableFixedJointLumping>true</disableFixedJointLumping>
         </gazebo>
         <xacro:if value="$(arg use_sim)">
             <!-- radar sim plugin -->
-            <gazebo reference="${radar_name}_link">
+            <gazebo reference="${name_space}_radar_link">
                 <material>Gazebo/FlatBlack</material>
                 <sensor type="ray" name="rplidar">
@@ -64,7 +60,7 @@
                     </ray>
                     <plugin name="gazebo_rplidar" filename="libgazebo_ros_laser.so">
-                        <robotNamespace>$(arg ns)</robotNamespace>
+                        <robotNamespace>${name_space}</robotNamespace>
                         <topicName>scan</topicName>
-                        <frameName>${radar_name}_link</frameName>
+                        <frameName>${name_space}_radar_link</frameName>
                     </plugin>
                 </sensor>

File: urdf/common/sct_mini_wheel.urdf.xacro (robot description, xacro)
@@ -2,7 +2,7 @@
 <robot xmlns:xacro="http://ros.org/wiki/xacro" name="scout_wheel">
     <xacro:macro name="sct_mini_wheel"
-                 params="prefix connected_to wheel_x_offset wheel_y_offset wheel_z_offset rotation_degree">
+                 params="prefix connected_to wheel_x_offset wheel_y_offset wheel_z_offset rotation_degree name_space">
         <!--  link  -->
-        <link name="${prefix}_wheel">
+        <link name="${name_space}_${prefix}_wheel">
             <visual>
                 <origin xyz="0 0 0" rpy="0 0 0"/>
@@ -30,5 +30,5 @@
             <dynamics damping="0.0" friction="0.01"/>
             <parent link="${connected_to}"/>
-            <child link="${prefix}_wheel"/>
+            <child link="${name_space}_${prefix}_wheel"/>
         </joint>
     </xacro:macro>

File: urdf/scout/chassis.urdf.xacro (robot description, xacro)
@@ -9,6 +9,6 @@
     <xacro:property name="wheel_base" value="0.463951"/>
     <xacro:property name="wheel_offset_z" value="-0.100998"/>
-    <xacro:macro name="chassis">
-        <link name="base_link">
+    <xacro:macro name="chassis" params="name_space:='scout'">
+        <link name="${name_space}_base_link">
             <visual>
                 <origin xyz="0 0 0" rpy="1.5707 0 -1.5707"/>
@@ -24,5 +24,5 @@
             </collision>
         </link>
-        <link name="inertial_link">
+        <link name="${name_space}_inertial_link">
             <inertial>
                 <mass value="50"/>
@@ -33,22 +33,26 @@
         <joint name="inertial_joint" type="fixed">
             <origin xyz="0 0 0" rpy="0 0 0"/>
-            <parent link="base_link"/>
-            <child link="inertial_link"/>
+            <parent link="${name_space}_base_link"/>
+            <child link="${name_space}_inertial_link"/>
         </joint>
-        <xacro:sct_mini_wheel prefix="left_front" connected_to="base_link"
+        <xacro:sct_mini_wheel prefix="left_front" connected_to="${name_space}_base_link"
                      wheel_x_offset="${wheel_base/2}" wheel_y_offset="${wheel_track/2}"
                      wheel_z_offset="${wheel_offset_z}" rotation_degree="${-pi/2}"
+                     name_space="${name_space}"
         />
-        <xacro:sct_mini_wheel prefix="right_front" connected_to="base_link"
+        <xacro:sct_mini_wheel prefix="right_front" connected_to="${name_space}_base_link"
                      wheel_x_offset="${wheel_base/2}" wheel_y_offset="${-wheel_track/2}"
                      wheel_z_offset="${wheel_offset_z}" rotation_degree="${pi/2}"
+                     name_space="${name_space}"
         />
-        <xacro:sct_mini_wheel prefix="left_back" connected_to="base_link"
+        <xacro:sct_mini_wheel prefix="left_back" connected_to="${name_space}_base_link"
                      wheel_x_offset="${-wheel_base/2}" wheel_y_offset="${wheel_track/2}"
                      wheel_z_offset="${wheel_offset_z}" rotation_degree="${-pi/2}"
+                     name_space="${name_space}"
         />
-        <xacro:sct_mini_wheel prefix="right_back" connected_to="base_link"
+        <xacro:sct_mini_wheel prefix="right_back" connected_to="${name_space}_base_link"
                      wheel_x_offset="${-wheel_base/2}" wheel_y_offset="${-wheel_track/2}"
                      wheel_z_offset="${wheel_offset_z}" rotation_degree="${pi/2}"
+                     name_space="${name_space}"
         />
         <xacro:wheel_transmission prefix="left_front" mechanical_reduction="1"/>

File: urdf/scout/scout_mini.urdf.xacro (robot description, xacro)
@@ -8,9 +8,9 @@
     <xacro:if value="$(arg load_chassis)">
         <xacro:include filename="$(find sct_description)/urdf/scout/chassis.urdf.xacro"/>
-        <xacro:chassis/>
+        <xacro:chassis name_space="$(arg robot_ns)"/>
     </xacro:if>
     <xacro:if value="$(arg load_radar)">
         <xacro:include filename="$(find sct_description)/urdf/common/radar.urdf.xacro"/>
-        <xacro:RADAR connected_to="base_link" radar_name="radar" use_sim="$(arg use_sim)" name_space="$(arg robot_ns)"
+        <xacro:RADAR connected_to="$(arg robot_ns)_base_link" use_sim="$(arg use_sim)" name_space="$(arg robot_ns)"
                      xyz="0.0 0.0 0.35"
                      rpy="0.0 0.0 0.0"/>

Commit message: change radar collision and range value in link label and gazebo/sensor/range label respectively.

File: urdf/common/radar.urdf.xacro (robot description, xacro)
@@ -18,7 +18,13 @@
                 <origin xyz="0.0 0.0 0.0" rpy="0.0 0.0 0.0"/>
             </visual>
+<!--            <collision>-->
+<!--                <geometry>-->
+<!--                    <cylinder radius="0.03" length="0.03"/>-->
+<!--                </geometry>-->
+<!--                <origin xyz="0.0 0.0 0.0" rpy="0.0 0.0 0.0"/>-->
+<!--            </collision>-->
             <collision>
                 <geometry>
-                    <cylinder radius="0.03" length="0.03"/>
+                    <cylinder radius="0.36" length="0.03"/>
                 </geometry>
                 <origin xyz="0.0 0.0 0.0" rpy="0.0 0.0 0.0"/>
@@ -49,5 +55,6 @@
                         </scan>
                         <range>
-                            <min>0.260</min>
+<!--                            <min>0.260</min>-->
+                            <min>0.370</min>
                             <max>7.5</max>
                             <resolution>0.015</resolution>

Commit message: First commit.

File: urdf/common/radar.urdf.xacro (robot description, xacro)
@@ -2,13 +2,13 @@
 <robot xmlns:xacro="http://www.ros.org/wiki/xacro" name="radar">
     <xacro:include filename="$(find sct_description)/urdf/common/inertia_utils.urdf.xacro"/>
-    <xacro:macro name="RADAR" params="connected_to use_sim name_space xyz:='0 0 0' rpy:='0 0 0' ">
+    <xacro:macro name="RADAR" params="connected_to use_sim xyz:='0 0 0' rpy:='0 0 0' ">
         <!-- Radar is fixed to the base link -->
-        <joint name="${name_space}_radar_joint" type="fixed">
+        <joint name="radar_joint" type="fixed">
             <origin xyz="${xyz}" rpy="${rpy}"/>
             <parent link="${connected_to}"/>
-            <child link="${name_space}_radar_link"/>
+            <child link="radar_link"/>
         </joint>
         <!-- Radar link -->
-        <link name="${name_space}_radar_link">
+        <link name="radar_link">
             <xacro:cylinder_inertial_matrix m="0.1" r="0.03" h="0.05"/>
             <visual>
@@ -39,5 +39,5 @@
         <xacro:if value="$(arg use_sim)">
             <!-- radar sim plugin -->
-            <gazebo reference="${name_space}_radar_link">
+            <gazebo reference="radar_link">
                 <material>Gazebo/FlatBlack</material>
                 <sensor type="ray" name="rplidar">
@@ -67,7 +67,7 @@
                     </ray>
                     <plugin name="gazebo_rplidar" filename="libgazebo_ros_laser.so">
-                        <robotNamespace>${name_space}</robotNamespace>
+                        <robotNamespace>/</robotNamespace>
                         <topicName>scan</topicName>
-                        <frameName>${name_space}_radar_link</frameName>
+                        <frameName>radar_link</frameName>
                     </plugin>
                 </sensor>

File: urdf/common/sct_mini_wheel.urdf.xacro (robot description, xacro)
@@ -2,7 +2,7 @@
 <robot xmlns:xacro="http://ros.org/wiki/xacro" name="scout_wheel">
     <xacro:macro name="sct_mini_wheel"
-                 params="prefix connected_to wheel_x_offset wheel_y_offset wheel_z_offset rotation_degree name_space">
+                 params="prefix connected_to wheel_x_offset wheel_y_offset wheel_z_offset rotation_degree ">
         <!--  link  -->
-        <link name="${name_space}_${prefix}_wheel">
+        <link name="${prefix}_wheel">
             <visual>
                 <origin xyz="0 0 0" rpy="0 0 0"/>
@@ -30,5 +30,5 @@
             <dynamics damping="0.0" friction="0.01"/>
             <parent link="${connected_to}"/>
-            <child link="${name_space}_${prefix}_wheel"/>
+            <child link="${prefix}_wheel"/>
         </joint>
     </xacro:macro>

File: urdf/scout/chassis.urdf.xacro (robot description, xacro)
@@ -9,6 +9,6 @@
     <xacro:property name="wheel_base" value="0.463951"/>
     <xacro:property name="wheel_offset_z" value="-0.100998"/>
-    <xacro:macro name="chassis" params="name_space:='scout'">
-        <link name="${name_space}_base_link">
+    <xacro:macro name="chassis" >
+        <link name="base_link">
             <visual>
                 <origin xyz="0 0 0" rpy="1.5707 0 -1.5707"/>
@@ -24,5 +24,5 @@
             </collision>
         </link>
-        <link name="${name_space}_inertial_link">
+        <link name="inertial_link">
             <inertial>
                 <mass value="50"/>
@@ -33,26 +33,22 @@
         <joint name="inertial_joint" type="fixed">
             <origin xyz="0 0 0" rpy="0 0 0"/>
-            <parent link="${name_space}_base_link"/>
-            <child link="${name_space}_inertial_link"/>
+            <parent link="base_link"/>
+            <child link="inertial_link"/>
         </joint>
-        <xacro:sct_mini_wheel prefix="left_front" connected_to="${name_space}_base_link"
+        <xacro:sct_mini_wheel prefix="left_front" connected_to="base_link"
                      wheel_x_offset="${wheel_base/2}" wheel_y_offset="${wheel_track/2}"
                      wheel_z_offset="${wheel_offset_z}" rotation_degree="${-pi/2}"
-                     name_space="${name_space}"
         />
-        <xacro:sct_mini_wheel prefix="right_front" connected_to="${name_space}_base_link"
+        <xacro:sct_mini_wheel prefix="right_front" connected_to="base_link"
                      wheel_x_offset="${wheel_base/2}" wheel_y_offset="${-wheel_track/2}"
                      wheel_z_offset="${wheel_offset_z}" rotation_degree="${pi/2}"
-                     name_space="${name_space}"
         />
-        <xacro:sct_mini_wheel prefix="left_back" connected_to="${name_space}_base_link"
+        <xacro:sct_mini_wheel prefix="left_back" connected_to="base_link"
                      wheel_x_offset="${-wheel_base/2}" wheel_y_offset="${wheel_track/2}"
                      wheel_z_offset="${wheel_offset_z}" rotation_degree="${-pi/2}"
-                     name_space="${name_space}"
         />
-        <xacro:sct_mini_wheel prefix="right_back" connected_to="${name_space}_base_link"
+        <xacro:sct_mini_wheel prefix="right_back" connected_to="base_link"
                      wheel_x_offset="${-wheel_base/2}" wheel_y_offset="${-wheel_track/2}"
                      wheel_z_offset="${wheel_offset_z}" rotation_degree="${pi/2}"
-                     name_space="${name_space}"
         />
         <xacro:wheel_transmission prefix="left_front" mechanical_reduction="1"/>

File: urdf/scout/scout_mini.urdf.xacro (robot description, xacro)
@@ -5,12 +5,12 @@
     <xacro:arg name="load_odom_sim" default="true"/>
     <xacro:arg name="use_sim" default="true"/>
-    <xacro:arg name="robot_ns" default="scout"/>
+    <xacro:arg name="robot_ns" default="/"/>
     <xacro:if value="$(arg load_chassis)">
         <xacro:include filename="$(find sct_description)/urdf/scout/chassis.urdf.xacro"/>
-        <xacro:chassis name_space="$(arg robot_ns)"/>
+        <xacro:chassis />
     </xacro:if>
     <xacro:if value="$(arg load_radar)">
         <xacro:include filename="$(find sct_description)/urdf/common/radar.urdf.xacro"/>
-        <xacro:RADAR connected_to="$(arg robot_ns)_base_link" use_sim="$(arg use_sim)" name_space="$(arg robot_ns)"
+        <xacro:RADAR connected_to="base_link" use_sim="$(arg use_sim)"
                      xyz="0.0 0.0 0.35"
                      rpy="0.0 0.0 0.0"/>

Commit message: Change multi robot navigation mode to single robot, main modify files including urdf and gazebo file.

File: urdf/common/radar.urdf.xacro (robot description, xacro)
@@ -1,6 +1,6 @@
 <?xml version="1.0" encoding="utf-8"?>
-<robot xmlns:xacro="http://www.ros.org/wiki/xacro" name="radar">
+<robot xmlns:xacro="http://www.ros.org/wiki/xacro" name="single_lidar">
     <xacro:include filename="$(find sct_description)/urdf/common/inertia_utils.urdf.xacro"/>
-    <xacro:macro name="RADAR" params="connected_to use_sim xyz:='0 0 0' rpy:='0 0 0' ">
+    <xacro:macro name="lidar" params="connected_to use_sim xyz:='0 0 0' rpy:='0 0 0' ">
         <!-- Radar is fixed to the base link -->
         <joint name="radar_joint" type="fixed">
@@ -18,10 +18,4 @@
                 <origin xyz="0.0 0.0 0.0" rpy="0.0 0.0 0.0"/>
             </visual>
-<!--            <collision>-->
-<!--                <geometry>-->
-<!--                    <cylinder radius="0.03" length="0.03"/>-->
-<!--                </geometry>-->
-<!--                <origin xyz="0.0 0.0 0.0" rpy="0.0 0.0 0.0"/>-->
-<!--            </collision>-->
             <collision>
                 <geometry>
@@ -55,5 +49,4 @@
                         </scan>
                         <range>
-<!--                            <min>0.260</min>-->
                             <min>0.370</min>
                             <max>50.0</max>

File: urdf/common/sct_mini_wheel.urdf.xacro (robot description, xacro)
@@ -2,5 +2,5 @@
 <robot xmlns:xacro="http://ros.org/wiki/xacro" name="scout_wheel">
     <xacro:macro name="sct_mini_wheel"
-                 params="prefix connected_to wheel_x_offset wheel_y_offset wheel_z_offset rotation_degree ">
+                 params="prefix connected_to wheel_x_offset wheel_y_offset wheel_z_offset rotation_degree">
         <!--  link  -->
         <link name="${prefix}_wheel">

File: urdf/scout/scout_mini.urdf.xacro (robot description, xacro)
@@ -2,25 +2,31 @@
 <robot xmlns:xacro="http://ros.org/wiki/xacro" name="scout">
     <xacro:arg name="load_chassis" default="true"/>
-    <xacro:arg name="load_radar" default="true"/>
+    <xacro:arg name="load_lidar" default="true"/>
+    <!-- select_lidar: radar or rs_lidar16 -->
+    <xacro:arg name="select_lidar" default="rs_lidar16"/>
     <xacro:arg name="load_odom_sim" default="true"/>
     <xacro:arg name="use_sim" default="true"/>
-    <xacro:arg name="robot_ns" default="/"/>
+    <xacro:arg name="gpu" default="true"/>
+    <xacro:property name="gpu" value="$(arg gpu)" />
     <xacro:if value="$(arg load_chassis)">
         <xacro:include filename="$(find sct_description)/urdf/scout/chassis.urdf.xacro"/>
         <xacro:chassis />
     </xacro:if>
-    <xacro:if value="$(arg load_radar)">
+    <xacro:if value="$(arg load_lidar)">
         <xacro:include filename="$(find sct_description)/urdf/common/radar.urdf.xacro"/>
-        <xacro:RADAR connected_to="base_link" use_sim="$(arg use_sim)"
+        <xacro:lidar connected_to="base_link" use_sim="$(arg use_sim)"
                      xyz="0.0 0.0 0.35"
                      rpy="0.0 0.0 0.0"/>
     </xacro:if>
+<!--    <xacro:include filename="$(find sct_description)/urdf/common/VLP-16.urdf.xacro"/>-->
+<!--    <xacro:VLP-16 parent="base_link" name="velodyne" topic="/velodyne_points" hz="10" samples="440" gpu="${gpu}">-->
+<!--        <origin xyz="0 0 0.4" rpy="0 0 0" />-->
+<!--    </xacro:VLP-16>-->
     <xacro:if value="$(arg use_sim)">
         <xacro:if value="$(arg load_odom_sim)">
-            <!-- odom sim plugin -->
             <gazebo>
                 <plugin name="sct_odom_sim" filename="libsct_odom_sim.so">
                     <publish_rate>50.0</publish_rate>
-                    <robot_namespace>$(arg robot_ns)</robot_namespace>
+                    <robot_namespace>/</robot_namespace>
                 </plugin>
             </gazebo>
@@ -28,5 +34,5 @@
         <gazebo>
             <plugin name="sct_ros_control" filename="libsct_robot_hw_sim.so">
-                <robotNamespace>$(arg robot_ns)</robotNamespace>
+                <robotNamespace>/</robotNamespace>
                 <robotSimType>sct_gazebo/SctRobotHWSim</robotSimType>
             </plugin>
