Commit message: Add cartographer navigation method and modify some multi robot to single robot.

File: urdf/common/VLP-16.urdf.xacro (robot description, xacro)
@@ -4,6 +4,6 @@
     <xacro:macro name="VLP-16" params="*origin parent:=base_link name:=velodyne
     topic:=/velodyne_points
-    hz:=10 lasers:=16 samples:=1875 collision_range:=0.3 min_range:=0.9 max_range:=130.0 noise:=0.008
-    min_angle:=-${M_PI} max_angle:=${M_PI} gpu:=false vis:=false ">
+    hz:=10 lasers:=16 samples:=1875 collision_range:=0.3 min_range:=0.5 max_range:=100.0 noise:=0.0
+    min_angle:=-${M_PI} max_angle:=${M_PI} gpu:=false vis:=true ">
         <joint name="${name}_base_mount_joint" type="fixed">
             <xacro:insert_block name="origin" />
@@ -55,86 +55,92 @@
         </link>
         <!-- Gazebo requires the velodyne_gazebo_plugins package -->
-        <gazebo reference="${name}">
-            <xacro:if value="${gpu}">
-                <sensor type="gpu_ray" name="${name}-VLP16">
-                    <pose>0 0 0 0 0 0</pose>
-                    <visualize>${vis}</visualize>
-                    <update_rate>${hz}</update_rate>
-                    <ray>
-                        <scan>
-                            <horizontal>
-                                <samples>${samples}</samples>
-                                <resolution>1</resolution>
-                                <min_angle>${min_angle}</min_angle>
-                                <max_angle>${max_angle}</max_angle>
-                            </horizontal>
-                            <vertical>
-                                <samples>${lasers}</samples>
-                                <resolution>1</resolution>
-                                <min_angle>-${15.0*M_PI/180.0}</min_angle>
-                                <max_angle> ${15.0*M_PI/180.0}</max_angle>
-                            </vertical>
-                        </scan>
-                        <range>
-                            <min>${collision_range}</min>
-                            <max>${max_range+1}</max>
-                            <resolution>0.001</resolution>
-                        </range>
-                        <noise>
-                            <type>gaussian</type>
-                            <mean>0.0</mean>
-                            <stddev>0.0</stddev>
-                        </noise>
-                    </ray>
-                    <plugin name="gazebo_ros_laser_controller" filename="libgazebo_ros_velodyne_gpu_laser.so">
-                        <topicName>${topic}</topicName>
-                        <frameName>${name}</frameName>
-                        <min_range>${min_range}</min_range>
-                        <max_range>${max_range}</max_range>
-                        <gaussianNoise>${noise}</gaussianNoise>
-                    </plugin>
-                </sensor>
-            </xacro:if>
-            <xacro:unless value="${gpu}">
-                <sensor type="ray" name="${name}-VLP16">
-                    <pose>0 0 0 0 0 0</pose>
-                    <visualize>${vis}</visualize>
-                    <update_rate>${hz}</update_rate>
-                    <ray>
-                        <scan>
-                            <horizontal>
-                                <samples>${samples}</samples>
-                                <resolution>1</resolution>
-                                <min_angle>${min_angle}</min_angle>
-                                <max_angle>${max_angle}</max_angle>
-                            </horizontal>
-                            <vertical>
-                                <samples>${lasers}</samples>
-                                <resolution>1</resolution>
-                                <min_angle>-${15.0*M_PI/180.0}</min_angle>
-                                <max_angle> ${15.0*M_PI/180.0}</max_angle>
-                            </vertical>
-                        </scan>
-                        <range>
-                            <min>${collision_range}</min>
-                            <max>${max_range+1}</max>
-                            <resolution>0.001</resolution>
-                        </range>
-                        <noise>
-                            <type>gaussian</type>
-                            <mean>0.0</mean>
-                            <stddev>0.0</stddev>
-                        </noise>
-                    </ray>
-                    <plugin name="gazebo_ros_laser_controller" filename="libgazebo_ros_velodyne_laser.so">
-                        <topicName>${topic}</topicName>
-                        <frameName>${name}</frameName>
-                        <min_range>${min_range}</min_range>
-                        <max_range>${max_range}</max_range>
-                        <gaussianNoise>${noise}</gaussianNoise>
-                    </plugin>
-                </sensor>
-            </xacro:unless>
-        </gazebo>
+<!--        <gazebo reference="${name}_base_scan_joint">-->
+<!--            <disableFixedJointLumping>true</disableFixedJointLumping>-->
+<!--        </gazebo>-->
+<!--        <gazebo reference="${name}_base_mount_joint">-->
+<!--            <disableFixedJointLumping>true</disableFixedJointLumping>-->
+<!--        </gazebo>-->
+<!--        <gazebo reference="${name}">-->
+<!--            <xacro:if value="${gpu}">-->
+<!--                <sensor type="gpu_ray" name="${name}-VLP16">-->
+<!--                    <pose>0 0 0 0 0 0</pose>-->
+<!--                    <visualize>${vis}</visualize>-->
+<!--                    <update_rate>${hz}</update_rate>-->
+<!--                    <ray>-->
+<!--                        <scan>-->
+<!--                            <horizontal>-->
+<!--                                <samples>${samples}</samples>-->
+<!--                                <resolution>1</resolution>-->
+<!--                                <min_angle>${min_angle}</min_angle>-->
+<!--                                <max_angle>${max_angle}</max_angle>-->
+<!--                            </horizontal>-->
+<!--                            <vertical>-->
+<!--                                <samples>${lasers}</samples>-->
+<!--                                <resolution>1</resolution>-->
+<!--                                <min_angle>-${15.0*M_PI/180.0}</min_angle>-->
+<!--                                <max_angle> ${15.0*M_PI/180.0}</max_angle>-->
+<!--                            </vertical>-->
+<!--                        </scan>-->
+<!--                        <range>-->
+<!--                            <min>${collision_range}</min>-->
+<!--                            <max>${max_range+1}</max>-->
+<!--                            <resolution>0.001</resolution>-->
+<!--                        </range>-->
+<!--                        <noise>-->
+<!--                            <type>gaussian</type>-->
+<!--                            <mean>0.0</mean>-->
+<!--                            <stddev>0.0</stddev>-->
+<!--                        </noise>-->
+<!--                    </ray>-->
+<!--                    <plugin name="gazebo_ros_laser_controller" filename="libgazebo_ros_velodyne_gpu_laser.so">-->
+<!--                        <topicName>${topic}</topicName>-->
+<!--                        <frameName>${name}</frameName>-->
+<!--                        <min_range>${min_range}</min_range>-->
+<!--                        <max_range>${max_range}</max_range>-->
+<!--                        <gaussianNoise>${noise}</gaussianNoise>-->
+<!--                    </plugin>-->
+<!--                </sensor>-->
+<!--            </xacro:if>-->
+<!--            <xacro:unless value="${gpu}">-->
+<!--                <sensor type="ray" name="${name}-VLP16">-->
+<!--                    <pose>0 0 0 0 0 0</pose>-->
+<!--                    <visualize>${vis}</visualize>-->
+<!--                    <update_rate>${hz}</update_rate>-->
+<!--                    <ray>-->
+<!--                        <scan>-->
+<!--                            <horizontal>-->
+<!--                                <samples>${samples}</samples>-->
+<!--                                <resolution>1</resolution>-->
+<!--                                <min_angle>${min_angle}</min_angle>-->
+<!--                                <max_angle>${max_angle}</max_angle>-->
+<!--                            </horizontal>-->
+<!--                            <vertical>-->
+<!--                                <samples>${lasers}</samples>-->
+<!--                                <resolution>1</resolution>-->
+<!--                                <min_angle>-${15.0*M_PI/180.0}</min_angle>-->
+<!--                                <max_angle> ${15.0*M_PI/180.0}</max_angle>-->
+<!--                            </vertical>-->
+<!--                        </scan>-->
+<!--                        <range>-->
+<!--                            <min>${collision_range}</min>-->
+<!--                            <max>${max_range+1}</max>-->
+<!--                            <resolution>0.001</resolution>-->
+<!--                        </range>-->
+<!--                        <noise>-->
+<!--                            <type>gaussian</type>-->
+<!--                            <mean>0.0</mean>-->
+<!--                            <stddev>0.0</stddev>-->
+<!--                        </noise>-->
+<!--                    </ray>-->
+<!--                    <plugin name="gazebo_ros_laser_controller" filename="libgazebo_ros_velodyne_laser.so">-->
+<!--                        <topicName>${topic}</topicName>-->
+<!--                        <frameName>${name}</frameName>-->
+<!--                        <min_range>${min_range}</min_range>-->
+<!--                        <max_range>${max_range}</max_range>-->
+<!--                        <gaussianNoise>${noise}</gaussianNoise>-->
+<!--                    </plugin>-->
+<!--                </sensor>-->
+<!--            </xacro:unless>-->
+<!--        </gazebo>-->
     </xacro:macro>
 </robot>

File: urdf/common/radar.urdf.xacro (robot description, xacro)
@@ -50,5 +50,5 @@
                         <range>
                             <min>0.370</min>
-                            <max>50.0</max>
+                            <max>30.0</max>
                             <resolution>0.015</resolution>
                         </range>

File: urdf/scout/scout_mini.urdf.xacro (robot description, xacro)
@@ -1,6 +1,8 @@
 <?xml version="1.0"?>
 <robot xmlns:xacro="http://ros.org/wiki/xacro" name="scout">
+    <xacro:property name="M_PI" value="3.1415926535897931" />
     <xacro:arg name="load_chassis" default="true"/>
     <xacro:arg name="load_lidar" default="true"/>
+    <xacro:arg name="load_imu" default="true"/>
     <!-- select_lidar: radar or rs_lidar16 -->
     <xacro:arg name="select_lidar" default="rs_lidar16"/>
@@ -13,23 +15,28 @@
         <xacro:chassis />
     </xacro:if>
-    <xacro:if value="$(arg load_lidar)">
-        <xacro:include filename="$(find sct_description)/urdf/common/radar.urdf.xacro"/>
-        <xacro:lidar connected_to="base_link" use_sim="$(arg use_sim)"
-                     xyz="0.0 0.0 0.35"
-                     rpy="0.0 0.0 0.0"/>
+<!--    <xacro:if value="$(arg load_lidar)">-->
+<!--        <xacro:include filename="$(find sct_description)/urdf/common/radar.urdf.xacro"/>-->
+<!--        <xacro:lidar connected_to="base_link" use_sim="$(arg use_sim)"-->
+<!--                     xyz="0.0 0.0 0.35"-->
+<!--                     rpy="0.0 0.0 0.0"/>-->
+<!--    </xacro:if>-->
+    <xacro:include filename="$(find sct_description)/urdf/common/VLP-16.urdf.xacro"/>
+    <xacro:VLP-16 parent="base_link" name="velodyne" topic="/velodyne_points" hz="10" samples="440" gpu="${gpu}">
+        <origin xyz="0 0 0.4" rpy="0 0 0" />
+    </xacro:VLP-16>
+    <xacro:if value="$(arg load_imu)">
+        <xacro:include filename="$(find sct_description)/urdf/common/imu.urdf.xacro"/>
+        <xacro:IMU connected_to="base_link" imu_name="imu" use_sim="$(arg use_sim)"
+                   xyz="0.0 0.0 0.35" rpy="0 0.0 0"/>
     </xacro:if>
-<!--    <xacro:include filename="$(find sct_description)/urdf/common/VLP-16.urdf.xacro"/>-->
-<!--    <xacro:VLP-16 parent="base_link" name="velodyne" topic="/velodyne_points" hz="10" samples="440" gpu="${gpu}">-->
-<!--        <origin xyz="0 0 0.4" rpy="0 0 0" />-->
-<!--    </xacro:VLP-16>-->
     <xacro:if value="$(arg use_sim)">
-        <xacro:if value="$(arg load_odom_sim)">
-            <gazebo>
-                <plugin name="sct_odom_sim" filename="libsct_odom_sim.so">
-                    <publish_rate>50.0</publish_rate>
-                    <robot_namespace>/</robot_namespace>
-                </plugin>
-            </gazebo>
-        </xacro:if>
+<!--        <xacro:if value="$(arg load_odom_sim)">-->
+<!--            <gazebo>-->
+<!--                <plugin name="sct_odom_sim" filename="libsct_odom_sim.so">-->
+<!--                    <publish_rate>50.0</publish_rate>-->
+<!--                    <robot_namespace>/</robot_namespace>-->
+<!--                </plugin>-->
+<!--            </gazebo>-->
+<!--        </xacro:if>-->
         <gazebo>
             <plugin name="sct_ros_control" filename="libsct_robot_hw_sim.so">
