Commit message: Modify a bug about sct_mini_wheel transmission and deleted relative files of location.

File: urdf/common/sct_mini_wheel.urdf.xacro (robot description, xacro)
@@ -1,6 +1,6 @@
 <?xml version="1.0"?>
 <robot xmlns:xacro="http://ros.org/wiki/xacro" name="scout_wheel">
-    <xacro:macro name="wheel"
-                 params="prefix connected_to wheel_x_offset wheel_y_offset wheel_z_offset rotation_degree max_effort max_velocity">
+    <xacro:macro name="sct_mini_wheel"
+                 params="prefix connected_to wheel_x_offset wheel_y_offset wheel_z_offset rotation_degree">
         <!--  link  -->
         <link name="${prefix}_wheel">
@@ -25,7 +25,7 @@
         <!--  joint  -->
         <joint name="${prefix}_wheel_joint" type="revolute">
-            <axis xyz="0 0 -1"/>
+            <axis xyz="0 0 1"/>
             <origin xyz="${wheel_x_offset} ${wheel_y_offset} ${wheel_offset_z}" rpy="${rotation_degree} 0 0"/>
-            <limit effort="${max_effort}" velocity="${max_velocity}" lower="-1e9" upper="1e9"/>
+            <limit effort="50" velocity="100" lower="-1e9" upper="1e9"/>
             <dynamics damping="0.0" friction="0.01"/>
             <parent link="${connected_to}"/>

File: urdf/scout/chassis.urdf.xacro (robot description, xacro)
@@ -1,4 +1,4 @@
 <robot xmlns:xacro="http://www.ros.org/wiki/xacro">
-    <xacro:include filename="$(find sct_description)/urdf/common/wheel.urdf.xacro"/>
+    <xacro:include filename="$(find sct_description)/urdf/common/sct_mini_wheel.urdf.xacro"/>
     <!-- https://upload.wikimedia.org/wikipedia/commons/5/52/Wheelbase_and_Track.png -->
     <xacro:property name="base_x_size" value="0.6200000"/>
@@ -36,28 +36,24 @@
             <child link="inertial_link"/>
         </joint>
-        <xacro:wheel prefix="left_front" connected_to="inertial_link"
+        <xacro:sct_mini_wheel prefix="left_front" connected_to="base_link"
                      wheel_x_offset="${wheel_base/2}" wheel_y_offset="${wheel_track/2}"
                      wheel_z_offset="${wheel_offset_z}" rotation_degree="${-pi/2}"
-                     max_effort="50" max_velocity="100"
         />
-        <xacro:wheel prefix="right_front" connected_to="inertial_link"
+        <xacro:sct_mini_wheel prefix="right_front" connected_to="base_link"
                      wheel_x_offset="${wheel_base/2}" wheel_y_offset="${-wheel_track/2}"
                      wheel_z_offset="${wheel_offset_z}" rotation_degree="${pi/2}"
-                     max_effort="50" max_velocity="100"
         />
-        <xacro:wheel prefix="left_back" connected_to="inertial_link"
+        <xacro:sct_mini_wheel prefix="left_back" connected_to="base_link"
                      wheel_x_offset="${-wheel_base/2}" wheel_y_offset="${wheel_track/2}"
                      wheel_z_offset="${wheel_offset_z}" rotation_degree="${-pi/2}"
-                     max_effort="50" max_velocity="100"
         />
-        <xacro:wheel prefix="right_back" connected_to="inertial_link"
+        <xacro:sct_mini_wheel prefix="right_back" connected_to="base_link"
                      wheel_x_offset="${-wheel_base/2}" wheel_y_offset="${-wheel_track/2}"
                      wheel_z_offset="${wheel_offset_z}" rotation_degree="${pi/2}"
-                     max_effort="50" max_velocity="100"
         />
         <xacro:wheel_transmission prefix="left_front" mechanical_reduction="1"/>
-        <xacro:wheel_transmission prefix="right_front" mechanical_reduction="1"/>
+        <xacro:wheel_transmission prefix="right_front" mechanical_reduction="-1"/>
         <xacro:wheel_transmission prefix="left_back" mechanical_reduction="1"/>
-        <xacro:wheel_transmission prefix="right_back" mechanical_reduction="1"/>
+        <xacro:wheel_transmission prefix="right_back" mechanical_reduction="-1"/>
     </xacro:macro>
 </robot>

File: urdf/scout/scout_mini.urdf.xacro (robot description, xacro)
@@ -1,20 +1,32 @@
 <?xml version="1.0"?>
-<robot xmlns:xacro="http://ros.org/wiki/xacro" name="scout1">
+<robot xmlns:xacro="http://ros.org/wiki/xacro" name="scout">
     <xacro:arg name="load_chassis" default="true"/>
-    <xacro:arg name="load_location" default="true"/>
+    <xacro:arg name="load_radar" default="true"/>
+    <xacro:arg name="load_odom_sim" default="true"/>
     <xacro:arg name="use_sim" default="true"/>
+    <xacro:arg name="robot_name" default="scout1"/>
     <xacro:if value="$(arg load_chassis)">
         <xacro:include filename="$(find sct_description)/urdf/scout/chassis.urdf.xacro"/>
         <xacro:chassis/>
     </xacro:if>
-    <xacro:if value="$(arg load_location)">
-        <xacro:include filename="$(find sct_description)/urdf/common/location.urdf.xacro"/>
-        <xacro:location connected_to="base_link" location_name="location" use_sim="$(arg use_sim)"
-                      xyz="0.0 0.0 0.0" rpy="0.0 0.0 0.0" />
+    <xacro:if value="$(arg load_radar)">
+        <xacro:include filename="$(find sct_description)/urdf/common/radar.urdf.xacro"/>
+        <xacro:RADAR connected_to="base_link" radar_name="radar" use_sim="$(arg use_sim)" name_space="$(arg robot_name)"
+                     xyz="0.0 0.0 0.35"
+                     rpy="0.0 0.0 0.0"/>
     </xacro:if>
     <xacro:if value="$(arg use_sim)">
+        <xacro:if value="$(arg load_odom_sim)">
+            <!-- odom sim plugin -->
+            <gazebo>
+                <plugin name="sct_odom_sim" filename="libsct_odom_sim.so">
+                    <publish_rate>50.0</publish_rate>
+                    <robot_namespace>$(arg robot_name)</robot_namespace>
+                </plugin>
+            </gazebo>
+        </xacro:if>
         <gazebo>
             <plugin name="sct_ros_control" filename="libsct_robot_hw_sim.so">
-                <robotNamespace>/</robotNamespace>
+                <robotNamespace>$(arg robot_name)</robotNamespace>
                 <robotSimType>sct_gazebo/SctRobotHWSim</robotSimType>
             </plugin>

Commit message: Add sct_chassis_controller using diff drive controller.

File: urdf/common/sct_mini_wheel.urdf.xacro (robot description, xacro)
@@ -2,5 +2,5 @@
 <robot xmlns:xacro="http://ros.org/wiki/xacro" name="scout_wheel">
     <xacro:macro name="sct_mini_wheel"
-                 params="prefix connected_to wheel_x_offset wheel_y_offset wheel_z_offset rotation_degree">
+                 params="prefix connected_to wheel_x_offset wheel_y_offset wheel_z_offset rotation_degree rotation_ori">
         <!--  link  -->
         <link name="${prefix}_wheel">
@@ -19,11 +19,11 @@
                 <origin xyz="0 0 0" rpy="0 0 0"/>
                 <geometry>
-                    <mesh filename="package://sct_description/meshes/common/wheel.dae"/>
+                    <cylinder radius="0.08" length="0.09"/>
                 </geometry>
             </collision>
         </link>
         <!--  joint  -->
-        <joint name="${prefix}_wheel_joint" type="revolute">
-            <axis xyz="0 0 1"/>
+        <joint name="${prefix}_wheel_joint" type="continuous">
+            <axis xyz="0 0 ${rotation_ori}"/>
             <origin xyz="${wheel_x_offset} ${wheel_y_offset} ${wheel_offset_z}" rpy="${rotation_degree} 0 0"/>
             <limit effort="50" velocity="100" lower="-1e9" upper="1e9"/>
@@ -37,9 +37,9 @@
             <type>transmission_interface/SimpleTransmission</type>
             <actuator name="${prefix}_wheel_motor">
-                <hardwareInterface>hardware_interface/EffortJointInterface</hardwareInterface>
+                <hardwareInterface>hardware_interface/VelocityJointInterface</hardwareInterface>
                 <mechanicalReduction>${mechanical_reduction}</mechanicalReduction>
             </actuator>
             <joint name="${prefix}_wheel_joint">
-                <hardwareInterface>hardware_interface/EffortJointInterface</hardwareInterface>
+                <hardwareInterface>hardware_interface/VelocityJointInterface</hardwareInterface>
             </joint>
         </transmission>

File: urdf/scout/chassis.urdf.xacro (robot description, xacro)
@@ -38,14 +38,14 @@
         <xacro:sct_mini_wheel prefix="left_front" connected_to="base_link"
                      wheel_x_offset="${wheel_base/2}" wheel_y_offset="${wheel_track/2}"
-                     wheel_z_offset="${wheel_offset_z}" rotation_degree="${-pi/2}" />
+                     wheel_z_offset="${wheel_offset_z}" rotation_degree="${-pi/2}" rotation_ori="${1}"/>
         <xacro:sct_mini_wheel prefix="left_rear" connected_to="base_link"
                               wheel_x_offset="${-wheel_base/2}" wheel_y_offset="${wheel_track/2}"
-                              wheel_z_offset="${wheel_offset_z}" rotation_degree="${-pi/2}" />
+                              wheel_z_offset="${wheel_offset_z}" rotation_degree="${-pi/2}" rotation_ori="${1}"/>
         <xacro:sct_mini_wheel prefix="right_front" connected_to="base_link"
                      wheel_x_offset="${wheel_base/2}" wheel_y_offset="${-wheel_track/2}"
-                     wheel_z_offset="${wheel_offset_z}" rotation_degree="${pi/2}" />
+                     wheel_z_offset="${wheel_offset_z}" rotation_degree="${pi/2}" rotation_ori="${-1}"/>
         <xacro:sct_mini_wheel prefix="right_rear" connected_to="base_link"
                      wheel_x_offset="${-wheel_base/2}" wheel_y_offset="${-wheel_track/2}"
-                     wheel_z_offset="${wheel_offset_z}" rotation_degree="${pi/2}" />
+                     wheel_z_offset="${wheel_offset_z}" rotation_degree="${pi/2}" rotation_ori="${-1}"/>
         <!-- those wheel transmission useless when don't use ros-control   -->
         <xacro:wheel_transmission prefix="left_front" mechanical_reduction="1"/>
@@ -53,26 +53,26 @@
         <xacro:wheel_transmission prefix="left_rear" mechanical_reduction="1"/>
         <xacro:wheel_transmission prefix="right_rear" mechanical_reduction="-1"/>
-        <xacro:if value="$(arg use_sim)">
-            <gazebo>
-                <plugin name="sct_chassis_sim" filename="libsct_chassis_sim.so">
-                    <updateRate>50.0</updateRate>
-                    <leftFrontJoint>left_front_wheel_joint</leftFrontJoint>
-                    <leftFrontTransmission>1.0</leftFrontTransmission>
-                    <rightFrontJoint>right_front_wheel_joint</rightFrontJoint>
-                    <rightFrontTransmission>-1.0</rightFrontTransmission>
-                    <leftRearJoint>left_rear_wheel_joint</leftRearJoint>
-                    <leftRearTransmission>1.0</leftRearTransmission>
-                    <rightRearJoint>right_rear_wheel_joint</rightRearJoint>
-                    <rightRearTransmission>-1.0</rightRearTransmission>
-                    <wheelTrack>${wheel_track}</wheelTrack>
-                    <wheelRadius>${wheel_radius}</wheelRadius>
-                    <torque>20</torque>
-                    <commandTopic>cmd_vel</commandTopic>
-                    <covariance_x>0.0001</covariance_x>
-                    <covariance_y>0.0001</covariance_y>
-                    <covariance_yaw>0.0001</covariance_yaw>
-                </plugin>
-            </gazebo>
-        </xacro:if>
+<!--        <xacro:if value="$(arg use_sim)">-->
+<!--            <gazebo>-->
+<!--                <plugin name="sct_chassis_sim" filename="libsct_chassis_sim.so">-->
+<!--                    <updateRate>50.0</updateRate>-->
+<!--                    <leftFrontJoint>left_front_wheel_joint</leftFrontJoint>-->
+<!--                    <leftFrontTransmission>1.0</leftFrontTransmission>-->
+<!--                    <rightFrontJoint>right_front_wheel_joint</rightFrontJoint>-->
+<!--                    <rightFrontTransmission>-1.0</rightFrontTransmission>-->
+<!--                    <leftRearJoint>left_rear_wheel_joint</leftRearJoint>-->
+<!--                    <leftRearTransmission>1.0</leftRearTransmission>-->
+<!--                    <rightRearJoint>right_rear_wheel_joint</rightRearJoint>-->
+<!--                    <rightRearTransmission>-1.0</rightRearTransmission>-->
+<!--                    <wheelTrack>${wheel_track}</wheelTrack>-->
+<!--                    <wheelRadius>${wheel_radius}</wheelRadius>-->
+<!--                    <torque>20</torque>-->
+<!--                    <commandTopic>cmd_vel</commandTopic>-->
+<!--                    <covariance_x>0.0001</covariance_x>-->
+<!--                    <covariance_y>0.0001</covariance_y>-->
+<!--                    <covariance_yaw>0.0001</covariance_yaw>-->
+<!--                </plugin>-->
+<!--            </gazebo>-->
+<!--        </xacro:if>-->
     </xacro:macro>
 </robot>

File: urdf/scout/scout_mini.urdf.xacro (robot description, xacro)
@@ -36,4 +36,9 @@
 <!--    </xacro:if>-->
     <xacro:if value="$(arg use_sim)">
+        <gazebo>
+            <plugin name="gazebo_ros_control" filename="libgazebo_ros_control.so">
+                <robotNamespace>/</robotNamespace>
+            </plugin>
+        </gazebo>
 <!--        <xacro:if value="$(arg load_odom_sim)">-->
 <!--            <gazebo>-->

Commit message: Add multi robot lauch.

File: urdf/common/sct_mini_wheel.urdf.xacro (robot description, xacro)
@@ -27,5 +27,5 @@
             <axis xyz="0 0 ${rotation_ori}"/>
             <origin xyz="${wheel_x_offset} ${wheel_y_offset} ${wheel_offset_z}" rpy="${rotation_degree} 0 0"/>
-            <limit effort="50" velocity="100" lower="-1e9" upper="1e9"/>
+<!--            <limit effort="30" velocity="50" lower="-1e9" upper="1e9"/>-->
             <dynamics damping="0.0" friction="0.01"/>
             <parent link="${connected_to}"/>

File: urdf/scout/chassis.urdf.xacro (robot description, xacro)
@@ -50,7 +50,7 @@
         <!-- those wheel transmission useless when don't use ros-control   -->
         <xacro:wheel_transmission prefix="left_front" mechanical_reduction="1"/>
-        <xacro:wheel_transmission prefix="right_front" mechanical_reduction="-1"/>
+        <xacro:wheel_transmission prefix="right_front" mechanical_reduction="1"/>
         <xacro:wheel_transmission prefix="left_rear" mechanical_reduction="1"/>
-        <xacro:wheel_transmission prefix="right_rear" mechanical_reduction="-1"/>
+        <xacro:wheel_transmission prefix="right_rear" mechanical_reduction="1"/>
 <!--        <xacro:if value="$(arg use_sim)">-->
 <!--            <gazebo>-->

File: urdf/scout/scout_mini.urdf.xacro (robot description, xacro)
@@ -18,5 +18,5 @@
     <xacro:if value="$(arg load_lidar)">
         <xacro:include filename="$(find sct_description)/urdf/common/os1_64.urdf.xacro"/>
-        <xacro:os1_64 connected_to="base_link" xyz="0.0 0.0 0.35" rpy="0.0 0.0 0.0"
+        <xacro:os1_64 connected_to="base_link" xyz="0.0 0.0 0.5" rpy="0.0 0.0 0.0"
                       use_sim="$(arg use_sim)" gpu="true"/>
     </xacro:if>
@@ -52,5 +52,5 @@
 <!--        <gazebo>-->
 <!--            <plugin name="sct_ros_control" filename="libsct_robot_hw_sim.so">-->
-<!--                <robotNamespace>/</robotNamespace>-->
+<!--                <robotNamespace>$(arg ns)</robotNamespace>-->
 <!--                <robotSimType>sct_gazebo/SctRobotHWSim</robotSimType>-->
 <!--            </plugin>-->
