Commit message: Update scout mini urdf.

File: urdf/common/os1_64.urdf.xacro (robot description, xacro)
@@ -40,5 +40,6 @@
         <origin xyz="0 0 0" rpy="0 0 0"/>
         <geometry>
-          <mesh filename="package://sct_description/meshes/common/${file_visual}.stl" />
+<!--          <mesh filename="package://sct_description/meshes/common/${file_visual}.stl" />-->
+          <mesh filename="package://sct_description/meshes/common/ouster_lidar.stl" scale="0.001 0.001 0.001"/>
         </geometry>
       </visual>

File: urdf/scout/chassis.urdf.xacro (robot description, xacro)
@@ -15,4 +15,16 @@
                 <geometry>
                     <mesh filename="package://sct_description/meshes/scout/base_link.dae"/>
+                </geometry>
+            </visual>
+<!--            <visual>-->
+<!--                <origin xyz="0 0 0" rpy="0.0 0.0 0.0"/>-->
+<!--                <geometry>-->
+<!--                    <mesh filename="package://sct_description/meshes/scout/base_link.stl" scale="0.001 0.001 0.001"/>-->
+<!--                </geometry>-->
+<!--            </visual>-->
+            <visual>
+                <origin xyz="0 0 0.15" rpy="0.0 0.0 0.0"/>
+                <geometry>
+                    <mesh filename="package://sct_description/meshes/scout/upper_shell.stl" scale="0.001 0.001 0.001"/>
                 </geometry>
             </visual>

File: urdf/scout/scout_mini.urdf.xacro (robot description, xacro)
@@ -18,5 +18,5 @@
     <xacro:if value="$(arg load_lidar)">
         <xacro:include filename="$(find sct_description)/urdf/common/os1_64.urdf.xacro"/>
-        <xacro:os1_64 connected_to="base_link" xyz="0.0 0.0 0.5" rpy="0.0 0.0 0.0"
+        <xacro:os1_64 connected_to="base_link" xyz="0.1349044 0.0 0.265" rpy="0.0 0.0 0.0"
                       use_sim="$(arg use_sim)" gpu="true"/>
     </xacro:if>
