Commit message: Build single-robot branch to test single navigation in ouster lidar.

File: urdf/scout/scout_mini.urdf.xacro (robot description, xacro)
@@ -15,14 +15,14 @@
         <xacro:chassis />
     </xacro:if>
-<!--    <xacro:if value="$(arg load_lidar)">-->
-<!--        <xacro:include filename="$(find sct_description)/urdf/common/radar.urdf.xacro"/>-->
-<!--        <xacro:lidar connected_to="base_link" use_sim="$(arg use_sim)"-->
-<!--                     xyz="0.0 0.0 0.35"-->
-<!--                     rpy="0.0 0.0 0.0"/>-->
-<!--    </xacro:if>-->
-    <xacro:include filename="$(find sct_description)/urdf/common/VLP-16.urdf.xacro"/>
-    <xacro:VLP-16 parent="base_link" name="velodyne" topic="/velodyne_points" hz="10" samples="440" gpu="${gpu}">
-        <origin xyz="0 0 0.4" rpy="0 0 0" />
-    </xacro:VLP-16>
+    <xacro:if value="$(arg load_lidar)">
+        <xacro:include filename="$(find sct_description)/urdf/common/radar.urdf.xacro"/>
+        <xacro:lidar connected_to="base_link" use_sim="$(arg use_sim)"
+                     xyz="0.0 0.0 0.35"
+                     rpy="0.0 0.0 0.0"/>
+    </xacro:if>
+<!--    <xacro:include filename="$(find sct_description)/urdf/common/VLP-16.urdf.xacro"/>-->
+<!--    <xacro:VLP-16 parent="base_link" name="velodyne" topic="/velodyne_points" hz="10" samples="440" gpu="${gpu}">-->
+<!--        <origin xyz="0 0 0.4" rpy="0 0 0" />-->
+<!--    </xacro:VLP-16>-->
     <xacro:if value="$(arg load_imu)">
         <xacro:include filename="$(find sct_description)/urdf/common/imu.urdf.xacro"/>
@@ -31,12 +31,12 @@
     </xacro:if>
     <xacro:if value="$(arg use_sim)">
-<!--        <xacro:if value="$(arg load_odom_sim)">-->
-<!--            <gazebo>-->
-<!--                <plugin name="sct_odom_sim" filename="libsct_odom_sim.so">-->
-<!--                    <publish_rate>50.0</publish_rate>-->
-<!--                    <robot_namespace>/</robot_namespace>-->
-<!--                </plugin>-->
-<!--            </gazebo>-->
-<!--        </xacro:if>-->
+        <xacro:if value="$(arg load_odom_sim)">
+            <gazebo>
+                <plugin name="sct_odom_sim" filename="libsct_odom_sim.so">
+                    <publish_rate>50.0</publish_rate>
+                    <robot_namespace>/</robot_namespace>
+                </plugin>
+            </gazebo>
+        </xacro:if>
         <gazebo>
             <plugin name="sct_ros_control" filename="libsct_robot_hw_sim.so">
