Commit message: Add scout mini chassis controller plugin of gazebo. .

File: urdf/scout/chassis.urdf.xacro (robot description, xacro)
@@ -9,5 +9,5 @@
     <xacro:property name="wheel_base" value="0.463951"/>
     <xacro:property name="wheel_offset_z" value="-0.100998"/>
-    <xacro:macro name="chassis" >
+    <xacro:macro name="chassis" params="use_sim:=false">
         <link name="base_link">
             <visual>
@@ -38,22 +38,42 @@
         <xacro:sct_mini_wheel prefix="left_front" connected_to="base_link"
                      wheel_x_offset="${wheel_base/2}" wheel_y_offset="${wheel_track/2}"
-                     wheel_z_offset="${wheel_offset_z}" rotation_degree="${-pi/2}"
-        />
+                     wheel_z_offset="${wheel_offset_z}" rotation_degree="${-pi/2}" />
+        <xacro:sct_mini_wheel prefix="left_rear" connected_to="base_link"
+                              wheel_x_offset="${-wheel_base/2}" wheel_y_offset="${wheel_track/2}"
+                              wheel_z_offset="${wheel_offset_z}" rotation_degree="${-pi/2}" />
         <xacro:sct_mini_wheel prefix="right_front" connected_to="base_link"
                      wheel_x_offset="${wheel_base/2}" wheel_y_offset="${-wheel_track/2}"
-                     wheel_z_offset="${wheel_offset_z}" rotation_degree="${pi/2}"
-        />
-        <xacro:sct_mini_wheel prefix="left_back" connected_to="base_link"
-                     wheel_x_offset="${-wheel_base/2}" wheel_y_offset="${wheel_track/2}"
-                     wheel_z_offset="${wheel_offset_z}" rotation_degree="${-pi/2}"
-        />
-        <xacro:sct_mini_wheel prefix="right_back" connected_to="base_link"
+                     wheel_z_offset="${wheel_offset_z}" rotation_degree="${pi/2}" />
+        <xacro:sct_mini_wheel prefix="right_rear" connected_to="base_link"
                      wheel_x_offset="${-wheel_base/2}" wheel_y_offset="${-wheel_track/2}"
-                     wheel_z_offset="${wheel_offset_z}" rotation_degree="${pi/2}"
-        />
+                     wheel_z_offset="${wheel_offset_z}" rotation_degree="${pi/2}" />
+        <!-- those wheel transmission useless when don't use ros-control   -->
         <xacro:wheel_transmission prefix="left_front" mechanical_reduction="1"/>
         <xacro:wheel_transmission prefix="right_front" mechanical_reduction="-1"/>
-        <xacro:wheel_transmission prefix="left_back" mechanical_reduction="1"/>
-        <xacro:wheel_transmission prefix="right_back" mechanical_reduction="-1"/>
+        <xacro:wheel_transmission prefix="left_rear" mechanical_reduction="1"/>
+        <xacro:wheel_transmission prefix="right_rear" mechanical_reduction="-1"/>
+        <xacro:if value="$(arg use_sim)">
+            <gazebo>
+                <plugin name="sct_chassis_sim" filename="libsct_chassis_sim.so">
+                    <robotNamespace>/</robotNamespace>
+                    <updateRate>50.0</updateRate>
+                    <leftFrontJoint>left_front_wheel_joint</leftFrontJoint>
+                    <leftFrontTransmission>1.0</leftFrontTransmission>
+                    <rightFrontJoint>right_front_wheel_joint</rightFrontJoint>
+                    <rightFrontTransmission>-1.0</rightFrontTransmission>
+                    <leftRearJoint>left_rear_wheel_joint</leftRearJoint>
+                    <leftRearTransmission>1.0</leftRearTransmission>
+                    <rightRearJoint>right_rear_wheel_joint</rightRearJoint>
+                    <rightRearTransmission>-1.0</rightRearTransmission>
+                    <wheelTrack>${wheel_track}</wheelTrack>
+                    <wheelRadius>${wheel_radius}</wheelRadius>
+                    <torque>30</torque>
+                    <commandTopic>cmd_vel</commandTopic>
+                    <covariance_x>0.0001</covariance_x>
+                    <covariance_y>0.0001</covariance_y>
+                    <covariance_yaw>0.0001</covariance_yaw>
+                </plugin>
+            </gazebo>
+        </xacro:if>
     </xacro:macro>
 </robot>

File: urdf/scout/scout_mini.urdf.xacro (robot description, xacro)
@@ -13,11 +13,10 @@
     <xacro:if value="$(arg load_chassis)">
         <xacro:include filename="$(find sct_description)/urdf/scout/chassis.urdf.xacro"/>
-        <xacro:chassis />
+        <xacro:chassis use_sim="$(arg use_sim)"/>
     </xacro:if>
     <xacro:if value="$(arg load_lidar)">
-        <xacro:include filename="$(find sct_description)/urdf/common/ouster_lidar.urdf.xacro"/>
-        <xacro:lidar connected_to="base_link" use_sim="$(arg use_sim)"
-                     xyz="0.0 0.0 0.35"
-                     rpy="0.0 0.0 0.0"/>
+        <xacro:include filename="$(find sct_description)/urdf/common/os1_64.urdf.xacro"/>
+        <xacro:os1_64 connected_to="base_link" xyz="0.0 0.0 0.35" rpy="0.0 0.0 0.0"
+                      use_sim="$(arg use_sim)" gpu="true"/>
     </xacro:if>
 <!--    <xacro:if value="$(arg load_lidar)">-->
@@ -37,18 +36,18 @@
 <!--    </xacro:if>-->
     <xacro:if value="$(arg use_sim)">
-        <xacro:if value="$(arg load_odom_sim)">
-            <gazebo>
-                <plugin name="sct_odom_sim" filename="libsct_odom_sim.so">
-                    <publish_rate>50.0</publish_rate>
-                    <robot_namespace>/</robot_namespace>
-                </plugin>
-            </gazebo>
-        </xacro:if>
-        <gazebo>
-            <plugin name="sct_ros_control" filename="libsct_robot_hw_sim.so">
-                <robotNamespace>/</robotNamespace>
-                <robotSimType>sct_gazebo/SctRobotHWSim</robotSimType>
-            </plugin>
-        </gazebo>
+<!--        <xacro:if value="$(arg load_odom_sim)">-->
+<!--            <gazebo>-->
+<!--                <plugin name="sct_odom_sim" filename="libsct_odom_sim.so">-->
+<!--                    <publish_rate>50.0</publish_rate>-->
+<!--                    <robot_namespace>/</robot_namespace>-->
+<!--                </plugin>-->
+<!--            </gazebo>-->
+<!--        </xacro:if>-->
+<!--        <gazebo>-->
+<!--            <plugin name="sct_ros_control" filename="libsct_robot_hw_sim.so">-->
+<!--                <robotNamespace>/</robotNamespace>-->
+<!--                <robotSimType>sct_gazebo/SctRobotHWSim</robotSimType>-->
+<!--            </plugin>-->
+<!--        </gazebo>-->
     </xacro:if>
 </robot>
